Commit message: urdf a bombar

File: p3dx_description/urdf/pioneer3dx.urdf (robot description, URDF)
Before this commit: robot pioneer3dx, 11 links, 10 joints
Links:
- link center_hubcap: geometry collision box size=0.00001 0.00001 0.00001; visual mesh filename=package://p3dx_description/meshes/center_hubcap.stl
- link center_wheel: mass 0.1 -> 1.0
- link front_sonar: geometry collision box size=0.00001 0.00001 0.00001; visual mesh filename=package://p3dx_description/meshes/front_sonar.stl
- link p3dx_left_hubcap: geometry collision box size=0.00001 0.00001 0.00001; visual mesh filename=package://p3dx_description/meshes/left_hubcap.stl
- link p3dx_right_hubcap: geometry collision box size=0.00001 0.00001 0.00001; visual mesh filename=package://p3dx_description/meshes/right_hubcap.stl
- link swivel: geometry collision box size=0.00001 0.00001 0.00001; visual mesh filename=package://p3dx_description/meshes/swivel.stl
Joints:
- joint base_swivel_joint: type continuous -> fixed
- joint lms100_joint: origin xyz=0.16 0 0.15 rpy=0 0 0 -> xyz=0.12 0 0.26 rpy=0 0 0
- joint swivel_hubcap_joint: type continuous -> fixed

File: p3dx_description/urdf/pioneer3dx.xacro (robot description, xacro)
@@ -16,10 +16,11 @@
 work original in ucs-ros-pkg.
  -->
-<robot name="pioneer3dx" xmlns:xacro="http://ros.org/wiki/xacro">
-  <!-- import all gazebo-customization elements, including gazebo colors -->
-  <xacro:include filename="$(find p3dx_description)/urdf/pioneer3dx.gazebo" />
-  <!-- import the pioneer 3dx's wheels -->
-  <xacro:include filename="$(find p3dx_description)/urdf/pioneer3dx_wheel.xacro" />
-  <!-- chassis -->
+<robot name="pioneer3dx"
+	xmlns:xacro="http://ros.org/wiki/xacro">
+	<!-- import all gazebo-customization elements, including gazebo colors -->
+	<xacro:include filename="$(find p3dx_description)/urdf/pioneer3dx.gazebo" />
+	<!-- import the pioneer 3dx's wheels -->
+	<xacro:include filename="$(find p3dx_description)/urdf/pioneer3dx_wheel.xacro" />
+	<!-- chassis -->
 	<link name="base_link">
 		<inertial>
@@ -29,12 +30,10 @@
 			<inertia ixx="1" ixy="0" ixz="0" iyy="1" iyz="0" izz="1" />
 		</inertial>
-		<visual name="base_visual">
+		<visual>
 			<origin xyz="-0.045 0 0.148" rpy="0 0 0" />
 			<geometry name="pioneer_geom">
 				<mesh filename="package://p3dx_description/meshes/chassis.stl" />
 			</geometry>
-			<material name="ChassisRed">
-				<color rgba="0.851 0.0 0.0 1.0" />
-			</material>
+			<material name="ChassisRed"></material>
 		</visual>
 		<collision>
@@ -45,5 +44,5 @@
 		</collision>
 	</link>
-  <!-- top_plate -->
+	<!-- top_plate -->
 	<link name="top_plate">
 		<inertial>
@@ -52,12 +51,10 @@
 			<inertia ixx="1" ixy="0" ixz="0" iyy="1" iyz="0" izz="1" />
 		</inertial>
-		<visual name="base_visual">
+		<visual>
 			<origin xyz="0 0 0" rpy="0 0 0" />
 			<geometry name="top_geom">
 				<mesh filename="package://p3dx_description/meshes/top.stl" />
 			</geometry>
-			<material name="TopBlack">
-				<color rgba="0.038 0.038 0.038 1.0" />
-			</material>
+			<material name="TopBlack"></material>
 		</visual>
 		<collision>
@@ -73,5 +70,5 @@
 		<child link="top_plate" />
 	</joint>
-  <!-- swivel -->
+	<!-- swivel -->
 	<link name="swivel">
 		<inertial>
@@ -80,21 +77,19 @@
 			<inertia ixx="0.01" ixy="0" ixz="0" iyy="0.01" iyz="0" izz="0.01" />
 		</inertial>
-		<visual name="base_visual">
+		<visual>
 			<origin xyz="0 0 0" rpy="0 0 0" />
 			<geometry name="pioneer_geom">
 				<mesh filename="package://p3dx_description/meshes/swivel.stl" />
 			</geometry>
-			<material name="swivel">
-				<color rgba="0.5 0.5 0.5 1" />
-			</material>
-		</visual>
-		<collision>
-			<origin xyz="0 0 0" rpy="0 0 0" />
-			<geometry>
-				<box size="0 0 0" />
-			</geometry>
-		</collision>
-	</link>
-	<joint name="base_swivel_joint" type="continuous">
+			<material name="swivel"></material>
+		</visual>
+		<collision>
+			<origin xyz="0 0 0" rpy="0 0 0" />
+			<geometry>
+				<box size="0.00001 0.00001 0.00001" />
+			</geometry>
+		</collision>
+	</link>
+	<joint name="base_swivel_joint" type="fixed">
 		<origin xyz="-0.185 0 0.055" rpy="0 0 0" />
 		<axis xyz="0 0 1" />
@@ -105,29 +100,26 @@
 		<child link="swivel" />
 	</joint>
-  <!-- center_hubcap -->
+	<!-- center_hubcap -->
 	<link name="center_hubcap">
 		<inertial>
 			<mass value="0.01" />
 			<origin xyz="0 0 0" />
-			<inertia ixx="0.012411765597" ixy="-0.000711733678" ixz="0.00050272983"
-				iyy="0.015218160428" iyz="-0.000004273467" izz="0.011763977943" />
-		</inertial>
-		<visual name="base_visual">
+			<inertia ixx="0.012411765597" ixy="-0.000711733678" ixz="0.00050272983" iyy="0.015218160428" iyz="-0.000004273467" izz="0.011763977943" />
+		</inertial>
+		<visual>
 			<origin xyz="0 0 0" rpy="0 0 0" />
 			<geometry name="pioneer_geom">
 				<mesh filename="package://p3dx_description/meshes/center_hubcap.stl" />
 			</geometry>
-			<material name="swivel">
-				<color rgba="0.5 0.5 0.5 1" />
-			</material>
-		</visual>
-		<collision>
-			<origin xyz="0 0 0" rpy="0 0 0" />
-			<geometry>
-				<box size="0 0 0" />
-			</geometry>
-		</collision>
-	</link>
-	<joint name="swivel_hubcap_joint" type="continuous">
+			<material name="swivel"></material>
+		</visual>
+		<collision>
+			<origin xyz="0 0 0" rpy="0 0 0" />
+			<geometry>
+				<box size="0.00001 0.00001 0.00001" />
+			</geometry>
+		</collision>
+	</link>
+	<joint name="swivel_hubcap_joint" type="fixed">
 		<origin xyz="-0.026 0 -0.016" rpy="0 0 0" />
 		<axis xyz="0 1 0" />
@@ -138,20 +130,17 @@
 		<child link="center_wheel" />
 	</joint>
-  <!-- center_wheel -->
+	<!-- center_wheel -->
 	<link name="center_wheel">
 		<inertial>
-			<mass value="0.1" />
-			<origin xyz="0 0 0" />
-			<inertia ixx="0.012411765597" ixy="-0.000711733678" ixz="0.00050272983"
-				iyy="0.015218160428" iyz="-0.000004273467" izz="0.011763977943" />
-		</inertial>
-		<visual name="base_visual">
+			<mass value="1.0" />
+			<origin xyz="0 0 0" />
+			<inertia ixx="0.012411765597" ixy="-0.000711733678" ixz="0.00050272983" iyy="0.015218160428" iyz="-0.000004273467" izz="0.011763977943" />
+		</inertial>
+		<visual>
 			<origin xyz="0 0 0" rpy="0 0 0" />
 			<geometry name="pioneer_geom">
 				<mesh filename="package://p3dx_description/meshes/center_wheel.stl" />
 			</geometry>
-			<material name="WheelBlack">
-				<color rgba="0.117 0.117 0.117 1" />
-			</material>
+			<material name="WheelBlack"></material>
 		</visual>
 		<collision>
@@ -167,7 +156,13 @@
 		<child link="center_hubcap"/>
 	</joint>
-	<xacro:p3dx_wheel suffix="left" parent="base_link" reflect="1"/>
-	<xacro:p3dx_wheel suffix="right" parent="base_link" reflect="-1"/>
-  <!-- front_sonar -->
+	<!-- End of Legacy for diff drive plugin
+	https://github.com/ros-simulation/gazebo_ros_pkgs/pull/707/files
+	"This setting assumes you have a old package, where the right and left wheel are changed to fix a former code issue\n"
+	"To get rid of this error just set <legacyMode> to false if you just created a new package.\n"
+	"To fix an old package you have to exchange left wheel by the right wheel.\n"
+	-->
+	<xacro:p3dx_wheel suffix="left" parent="base_link" reflect="-1"/>
+	<xacro:p3dx_wheel suffix="right" parent="base_link" reflect="1"/>
+	<!-- front_sonar -->
 	<link name="front_sonar">
 		<inertial>
@@ -176,17 +171,15 @@
 			<inertia ixx="1" ixy="0" ixz="0" iyy="1" iyz="0" izz="1" />
 		</inertial>
-		<visual name="front_sonar_vis">
+		<visual>
 			<origin rpy="0 0 0" xyz="0 0 0" />
 			<geometry name="pioneer_geom">
 				<mesh filename="package://p3dx_description/meshes/front_sonar.stl" />
 			</geometry>
-			<material name="SonarYellow">
-				<color rgba="0.715 0.583 0.210 1.0" />
-			</material>
+			<material name="SonarYellow"></material>
 		</visual>
 		<collision>
 			<origin rpy="0 0 0" xyz="0 0 0" />
 			<geometry>
-				<box size="0 0 0" />
+				<box size="0.00001 0.00001 0.00001" />
 			</geometry>
 		</collision>
@@ -219,5 +212,5 @@
 	<joint name="lms100_joint" type="fixed">
 		<axis xyz="0 1 0" />
-		<origin xyz="0.16 0 0.15" rpy="0 0 0" />
+		<origin xyz="0.12 0 0.26" rpy="0 0 0" />
 		<parent link="base_link" />
 		<child link="lms100" />
